File: conception/PANEL_LED_HARDWARE/PANEL_LED_HARDWARE.kicad_sch (KiCad schematic)
At the start: 93 parts, among them J1 PWR, J2 Connector to pannel led, Q3 Q12MHz/20pF/30ppm/2P/HC-49SM(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, Q4 BC817-40(SOT23), Q5 BC817-40(SOT23), U1 SY8089AAAC(SOT23-5), U10 BAT54C(SOT23-3), U2 LM2576T-5, U3 ESP32-WROOM-32D-4MB, U4 LAN8710A-EZC(QFN32)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

Commit message: Update schematic
New ref ( LMR51430 ) for the 24/5V converter
Add package for alim and panel connecter
Parts:
- removed BUT1: T1107A(6x3,8x2,5MM), OLIMEX_Buttons-FP:T1107A(6x3,8x2,5MM), symbol ESP32-EVB_Rev_H:SIDE_WTCM-TR(3x4)
- removed C4: 100uF, symbol Device:C_Polarized_Small_US
- removed C41, C51: 10uF, symbol Device:C_Polarized_Small_US
- removed C5: 1000uF, symbol Device:C_Polarized_Small_US
- removed D1: 1N5822, Diode_THT:D_DO-201AD_P15.24mm_Horizontal, symbol Diode:1N5822
- removed EXT1: NA(HN2x20), OLIMEX_Connectors-FP:HN2x20, symbol ESP32-EVB_Rev_H:BH40S
- removed R14: 220R/R0603, OLIMEX_RLC-FP:R_0603_5MIL_DWS, symbol ESP32-EVB_Rev_H:R
- removed R45: 10k/R0603, OLIMEX_RLC-FP:R_0603_5MIL_DWS, symbol ESP32-EVB_Rev_H:R
- removed R46: NA/R0603, OLIMEX_RLC-FP:R_0603_5MIL_DWS, symbol ESP32-EVB_Rev_H:R
- removed U2: LM2576T-5, Package_TO_SOT_THT:TO-220-5_Vertical, symbol Regulator_Switching:LM2576T-5
- removed U6: LD1085V50, Package_TO_SOT_THT:TO-220-3_Vertical, symbol Regulator_Linear:LD1086V-DG
- added C4: 2.2uF, OLIMEX_RLC-FP:C_0603_5MIL_DWS, symbol ESP32-EVB_Rev_H:C
- added C5: 44uF, OLIMEX_RLC-FP:C_0603_5MIL_DWS, symbol ESP32-EVB_Rev_H:C
- added C6: 0.1uF, OLIMEX_RLC-FP:C_0603_5MIL_DWS, symbol ESP32-EVB_Rev_H:C
- added R1: 100k, OLIMEX_RLC-FP:R_0603_5MIL_DWS, symbol ESP32-EVB_Rev_H:R
- added R2: 13.7k, OLIMEX_RLC-FP:R_0603_5MIL_DWS, symbol ESP32-EVB_Rev_H:R
- added U1: LMR51430, symbol New_Library:LMR51430
- J1: footprint (none) -> PANEL_LED:BORNIER_2P
- J2: footprint (none) -> PANEL_LED:PANEL_CONNECTOR
- L1: value 100uH -> 6.8uH
Connections:
- net GND: now also C4.2, C5.2, R2.2, U1.1 (GND)
- net Vin +24V: now also C4.1, U1.3 (VIN), U1.5 (EN)
- net at D6.2 (A), FET1.1, L1.2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: now also C5.1, R1.1
- net at L1.1: now also C6.2, U1.2 (SW)
- new net: C6.1, U1.6 (CB)
- new net: R1.2, R2.1, U1.4 (FB)
Other:
- note added: "RESET"
- note removed: "Buttons"
- moved on the sheet: C1, C2, C3, C6, C7, D2, D4, D6, FET1, J1, J2, L1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

Commit message: Update hardware add latch
Parts:
- added C10: 2.2uF, OLIMEX_RLC-FP:C_0603_5MIL_DWS, symbol ESP32-EVB_Rev_H:C
- added C20: 44uF, OLIMEX_RLC-FP:C_0603_5MIL_DWS, symbol ESP32-EVB_Rev_H:C
- added C9: 0.1uF, OLIMEX_RLC-FP:C_0603_5MIL_DWS, symbol ESP32-EVB_Rev_H:C
- added J2: PWR_TO_LED, PANEL_LED:BORNIER_2P, symbol Connector_Generic:Conn_01x02
- added J4: PWR, PANEL_LED:BORNIER_2P, symbol Connector_Generic:Conn_01x02
- added L8: 6.8uH, OLIMEX_RLC-FP:L_0805_5MIL_DWS, symbol ESP32-EVB_Rev_H:L
- added R20: 13.7k, OLIMEX_RLC-FP:R_0603_5MIL_DWS, symbol ESP32-EVB_Rev_H:R
- added R52: 100k, OLIMEX_RLC-FP:R_0603_5MIL_DWS, symbol ESP32-EVB_Rev_H:R
- added U12: 74HC374, symbol 74xx:74HC374
- added U7: LMR51430, PANEL_LED:LMR51430, symbol New_Library:LMR51430
- U1: footprint (none) -> PANEL_LED:LMR51430
- renumbered J2 to J3, U1 to U2
Connections:
- net PANNEL_LAT is gone; now on net PANEL_LAT: J3.14
- net +5V: now also U12.20 (VCC)
- net GND: now also C10.2, C20.2, J2.1 (Pin_1), J4.1 (Pin_1), R20.2, U12.1 (OE), U12.10 (GND), U7.1 (GND)
- net PANEL_A: now also U12.9 (O3)
- net PANEL_B: now also U12.12 (O4)
- net PANEL_B1: now also U3.29 (GPIO5/VSPICS0/HS1_DATA6/EMAC_RX_CLK), U12.14 (D5)
- net PANEL_B2: now also U3.16 (GPIO13/ADC2_CH4/TOUCH4/RTC_GPIO14/MTCK/HSPID/HS2_DATA3/SD_DATA3/EMAC_RX_ER)
- net PANEL_C: now also U12.15 (O5)
- net PANEL_CLK: now also U3.27 (GPIO16/HS1_DATA4/U2RXD/EMAC_CLK_OUT)
- net PANEL_G1: now also U3.23 (GPIO15/ADC2_CH3/TOUCH3/MTDO/HSPICS0/RTC_GPIO13/HS2_CMD/SD_CMD/EMAC_RXD3), U12.13 (D4)
- net PANEL_G2: now also U3.14 (GPIO12/ADC2_CH5/TOUCH5/RTC_GPIO15/MTDI/HSPIQ/HS2_DATA2/SD_DATA2/EMAC_TXD3), U12.17 (D6), U12.18 (D7)
- net PANEL_R1: now also U3.28 (GPIO17/HS1_DATA5/U2TXD/EMAC_CLK_OUT_180), U12.7 (D2), U12.8 (D3)
- net PANEL_R2: now also U3.13 (GPIO14/ADC2_CH6/TOUCH6/RTC_GPIO16/MTMS/HSPICLK/HS2_CLK/SD_CLK/EMAC_TXD2), U12.3 (D0), U12.4 (D1)
- net Vin +24V: now also C10.1, J4.2 (Pin_2), U7.3 (VIN), U7.5 (EN)
- net 5V panel 1: now reaches C5.1, D6.2 (A), FET1.1, L1.2, R1.1, R30.1
- net 5V panel 1: now also C20.1, J2.2 (Pin_2), L8.2, R52.1
- net PANEL_LAT: now reaches U3.26 (GPIO4/ADC2_CH0/TOUCH0/RTC_GPIO10/HSPIHD/HS2_DATA1/SD_DATA1/EMAC_TX_ER)
- net PANEL_LAT: now also U12.11 (Cp)
- new net: C9.2, L8.1, U7.2 (SW)
- new net: R20.1, R52.2, U7.4 (FB)
- new net: C9.1, U7.6 (CB)
- new net PANEL_D: U12.5 (O1)
- new net PANEL_E: U12.16 (O6)
Other:
- note added: "PANNEL LED Connections"
- note removed: "Connector PANNEL LED"
- moved on the sheet: C1, C2, C3, C4, C5, C6, C7, D2, D4, D6, FET1, J1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

Commit message: Update hardware to connect daugther board
Parts:
- removed C11, C13, C14, C15, C17, C24: 100nF/50V/20%/Y5V/C0603, OLIMEX_RLC-FP:C_0603_5MIL_DWS, symbol ESP32-EVB_Rev_H:C
- removed C12, C23, C29, C8, C9: 22uF/6.3V/20%/X5R/C0603, OLIMEX_RLC-FP:C_0603_5MIL_DWS, symbol ESP32-EVB_Rev_H:C
- removed C16: 2.2uF/6.3V/10%/X5R/C0603, OLIMEX_RLC-FP:C_0603_5MIL_DWS, symbol ESP32-EVB_Rev_H:C
- removed C18: NA(10uF/6.3V/20%/X5R/C0603), OLIMEX_RLC-FP:C_0603_5MIL_DWS, symbol ESP32-EVB_Rev_H:C
- removed C19: 1nF/2000V/10%/X7R/C1206, OLIMEX_RLC-FP:C_1206_5MIL_DWS_ISO, symbol ESP32-EVB_Rev_H:C
- removed C20: NA(1nF/2000V/10%/X7R/C1206), OLIMEX_RLC-FP:C_1206_5MIL_DWS_ISO, symbol ESP32-EVB_Rev_H:C
- removed C21, C22: 27pF/50V/5%/C0G/C0603, OLIMEX_RLC-FP:C_0603_5MIL_DWS, symbol ESP32-EVB_Rev_H:C
- removed C28: 470nF/16V/10%/X7R/C0603, OLIMEX_RLC-FP:C_0603_5MIL_DWS, symbol ESP32-EVB_Rev_H:C
- removed CR1: Q50MHz/25ppm/3V/4P/5x3.2mm, OLIMEX_Crystal-FP:5032-4P_HCX-3S, symbol ESP32-EVB_Rev_H:Oscillator-100MHZ_TXC-7W
- removed D6: 1N5822/SS34/SMA, OLIMEX_Diodes-FP:SMA-KA, symbol ESP32-EVB_Rev_H:D_Schottky
- removed D7, D8: 1N5819S4(SOD-123), OLIMEX_Diodes-FP:SOD-123_1C-2A_KA, symbol ESP32-EVB_Rev_H:D_Schottky_Small
- removed FET1, FET3: WPM2015-3/TR, OLIMEX_Transistors-FP:SOT23, symbol ESP32-EVB_Rev_H:P-MOS+DIOD
- removed FET4: BSS138, OLIMEX_Transistors-FP:SOT23, symbol ESP32-EVB_Rev_H:N-MOS+DIOD
- removed L3: FB0805/600R/2A, OLIMEX_RLC-FP:L_0805_5MIL_DWS, symbol ESP32-EVB_Rev_H:L
- removed L5: NA(FB0805/600R/2A), OLIMEX_RLC-FP:L_0805_5MIL_DWS, symbol ESP32-EVB_Rev_H:L
- removed LAN1: RJLD-060TC1(LPJ4013EDNL), OLIMEX_Connectors-FP:RJLBC-060TC1, symbol ESP32-EVB_Rev_H:RJLBC-060TC1_GND
- removed PHY_RST1: Opened, OLIMEX_Jumpers-FP:SJ, symbol ESP32-EVB_Rev_H:SJ
- removed Q3: Q12MHz/20pF/30ppm/2P/HC-49SM(SMD), OLIMEX_Crystal-FP:Q_49U3HMS, symbol ESP32-EVB_Rev_H:Crystal
- removed Q4, Q5: BC817-40(SOT23), OLIMEX_Transistors-FP:SOT23, symbol ESP32-EVB_Rev_H:Q_NPN_BEC
- removed R24: 470k/R0603, OLIMEX_RLC-FP:R_0603_5MIL_DWS, symbol ESP32-EVB_Rev_H:R
- removed R25: 0R(board_mounted), OLIMEX_RLC-FP:0R_0603, symbol ESP32-EVB_Rev_H:R
- removed R26, R27, R37: 220R/R0603, OLIMEX_RLC-FP:R_0603_5MIL_DWS, symbol ESP32-EVB_Rev_H:R
- removed R28, R31, R32, R33: 49.9R/1%/R0603, OLIMEX_RLC-FP:R_0603_5MIL_DWS, symbol ESP32-EVB_Rev_H:R
- removed R30, R34, R35, R38, R40, R51: 10k/R0603, OLIMEX_RLC-FP:R_0603_5MIL_DWS, symbol ESP32-EVB_Rev_H:R
- removed R36: 10R/R0603, OLIMEX_RLC-FP:R_0603_5MIL_DWS, symbol ESP32-EVB_Rev_H:R
- removed R39: 12.1k/1%/R0603, OLIMEX_RLC-FP:R_0603_5MIL_DWS, symbol ESP32-EVB_Rev_H:R
- removed R41, R42, R50: 1k/R0603, OLIMEX_RLC-FP:R_0603_5MIL_DWS, symbol ESP32-EVB_Rev_H:R
- removed R44, R54: NA/R0603, OLIMEX_RLC-FP:R_0603_5MIL_DWS, symbol ESP32-EVB_Rev_H:R
- removed R57: NA(1k/R0603), OLIMEX_RLC-FP:R_0603_5MIL_DWS, symbol ESP32-EVB_Rev_H:R
- removed RM2, RM3: RA1206_(4X0603)_4B8_2.2k, OLIMEX_RLC-FP:R_MATRIX_4, symbol ESP32-EVB_Rev_H:RA1206_(4x0603)_4B8_Smashed
- removed RST1: T1107A(6x3,8x2,5MM), OLIMEX_Buttons-FP:T1107A(6x3,8x2,5MM), symbol ESP32-EVB_Rev_H:SIDE_WTCM-TR(3x4)
- removed U10, U9: BAT54C(SOT23-3), OLIMEX_Diodes-FP:SOT23-3, symbol ESP32-EVB_Rev_H:BAT54C(SOT23-3)
- removed U3: ESP32-WROOM-32D-4MB, OLIMEX_Cases-FP:ESP-WROOM-32_MODULE, symbol ESP32-EVB_Rev_H:ESP-WROOM-32
- removed U4: LAN8710A-EZC(QFN32), OLIMEX_IC-FP:QFN32_EP(33)_5.00x5.00x0.90mm_Pitch_0.50mm, symbol ESP32-EVB_Rev_H:LAN8710A-EZC(QFN32)
- removed U5: CH340T(SSOP20W), OLIMEX_IC-FP:SSOP-20W, symbol ESP32-EVB_Rev_H:CH340T(SSOP20W)
- removed U8: NCP303LSN27T1G(SOT-23-5), OLIMEX_IC-FP:SOT-23-5, symbol ESP32-EVB_Rev_H:BD5230G-TR(SSOP5_SOT-23-5)
- removed USB-UART1: MISB-SWMM-5B-LF(USB_MICRO), OLIMEX_Connectors-FP:USB-MICRO_MISB-SWMM-5B_LF, symbol ESP32-EVB_Rev_H:USB-MINI
- added J8: EXT PIN, symbol Connector:Conn_01x20_Female
Connections:
- net +3V3: now also J8.1 (Pin_1), J8.20 (Pin_20)
- net +5V: now also C5.1, J2.2 (Pin_2), L1.2, R1.1
- net ESP_EN: now also J8.3 (Pin_3)
- net GND: now also J8.19 (Pin_19), J8.2 (Pin_2)
- removed net 5V panel 1: C20.1, C5.1, J2.2 (Pin_2), L1.2, L8.2, R1.1, R52.1
- net PANEL_B1 renamed GPIO12\PANEL_B1
- net GPIO12\PANEL_B1: now also J8.7 (Pin_7)
- net PANEL_B2 renamed GPIO13\PANEL_B2
- net GPIO13\PANEL_B2: now also J8.8 (Pin_8)
- net PANEL_CLK renamed GPI016\PANEL_CLK
- net GPI016\PANEL_CLK: now also J8.11 (Pin_11)
- net PANEL_G1 renamed GPIO14\PANEL_G1
- net GPIO14\PANEL_G1: now also J8.9 (Pin_9)
- net PANEL_G2 renamed GPIO15\PANEL_G2
- net GPIO15\PANEL_G2: now also J8.10 (Pin_10)
- net PANEL_LAT renamed GPIO4\PANEL_LAT
- net GPIO4\PANEL_LAT: now also J8.6 (Pin_6)
- net PANEL_OE renamed GPI032\PANEL_OE
- net GPI032\PANEL_OE: now also J8.13 (Pin_13)
- net PANEL_R1 renamed GPI05\PANEL_R1
- net GPI05\PANEL_R1: now also J8.4 (Pin_4)
- net PANEL_R2 renamed GPIO17\PANEL_R2
- net GPIO17\PANEL_R2: now also J8.12 (Pin_12)
- new net: C20.1, L8.2, R52.1
- new net GPI033: J8.14 (Pin_14)
- new net GPI34: J8.15 (Pin_15)
- new net GPI35: J8.16 (Pin_16)
- new net GPI36: J8.17 (Pin_17)
- new net GPI39: J8.18 (Pin_18)
- new net GPIO2\HS2_DATA0: J8.5 (Pin_5)
- no-connect marks 12 -> 0
Other:
- note added: "Extension"
- note removed: "+5V_Only!!!"
- note removed: "0"
- note removed: "1"
- note removed: "Auto program"
- note removed: "CD"
- note removed: "DTR RTS->EN IO0"
- note removed: "ESP-WROOM-32 MODULE"
- note removed: "Ethernet"
- note removed: "In RMII Mode"
- note removed: "RESET"
- note removed: "The PHY is setted up as follows: MODE: All capable(10/100Base) -Auto-negotiation enabled -RMII Configuration -SMI address: 0x00"
- note removed: "USB to UART"
- note removed: "tD2 ≈ RD * CD RD = 1M Ohm -> typiclally CD = 470nF -> selected then: tD2 approx. 470ms"
- moved on the sheet: C1, C10, C2, C20, C3, C4, C5, C6, C7, C9, D2, D4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
